File: Menorah.sch (EAGLE design)
At the start: 0 parts

Commit message: design finished
Parts:
- added C1: 100uF, rcl:C-USC1808
- added G1: CR2032V, battery:CR2032V
- added IC1: (no value), linear:1AMP_P7+4D
- added LED1, LED2, LED3, LED4, LED5, LED6, LED7, LED8, LED9: (no value), led:LEDP-LCC-4
- added R1, R2, R3, R4, R5, R6, R7, R8, R9: (no value), rcl:R-US_R0805
- added R10: 10M, rcl:R-US_R0805
- added R11: 50k, rcl:R-US_R0805
- added R12: 100k, rcl:R-US_R0805
- added S1, S2, S3, S4, S5, S6, S7, S8, S9: 2P2T, switch:2P2T
- added S10: RDT1034, switch:RDT1034
Connections:
- new net N$1: LED1.A, R1.2
- new net N$10: R1.1, S1.3.2
- new net N$11: R2.1, S2.3.2
- new net N$12: R3.1, S3.3.2
- new net N$13: R4.1, S4.3.2
- new net N$14: R5.1, S5.3.2
- new net N$15: R6.1, S6.3.2
- new net N$16: R7.1, S7.3.2
- new net N$17: R8.1, S8.3.2
- new net N$18: R9.1, S9.3.2
- new net N$19: IC1.-IN, R11.1, R12.2
- new net N$2: LED2.A, R2.2
- new net N$20: C1.1, IC1.+IN, R10.2, S10.B
- new net N$21: IC1.OUT, S1.2.1
- new net N$23: S1.2.2, S2.2.1
- new net N$24: S2.2.2, S3.2.1
- new net N$25: S3.2.2, S4.2.1
- new net N$26: S4.2.2, S5.2.1
- new net N$27: S5.2.2, S6.2.1
- new net N$28: S6.2.2, S7.2.1
- new net N$29: S7.2.2, S8.2.1
- new net N$3: LED3.A, R3.2
- new net N$30: S8.2.2, S9.2.1
- new net N$4: LED4.A, R4.2
- new net N$5: LED5.A, R5.2
- new net N$6: LED6.A, R6.2
- new net N$7: LED7.A, R7.2
- new net N$8: LED8.A, R8.2
- new net N$9: LED9.A, R9.2
- new net PE: C1.2, G1.-, IC1.V-, LED1.C, LED2.C, LED3.C, LED4.C, LED5.C, LED6.C, LED7.C, LED8.C, LED9.C, R10.1, R11.2
- new net VCC: G1.+, IC1.V+, R12.1, S10.A, S10.A1
