File: Menorah.brd (EAGLE design)
At the start: 100 x 80 mm, 34 parts

Commit message: replaced dpdt switch
Parts:
- S1, S2, S3, S4, S5, S6, S7, S8, S9: value 2P2T -> SWITCH-DPDT; device switch:2P2T -> Menorah:JS202011SCQN
Connections:
- net N$10: now also S1.3; no longer S1.3.2
- net N$11: now also S2.3; no longer S2.3.2
- net N$12: now also S3.3; no longer S3.3.2
- net N$13: now also S4.3; no longer S4.3.2
- net N$14: now also S5.3; no longer S5.3.2
- net N$15: now also S6.3; no longer S6.3.2
- net N$16: now also S7.3; no longer S7.3.2
- net N$17: now also S8.3; no longer S8.3.2
- net N$18: now also S9.3; no longer S9.3.2
- net N$21: now also S1.5; no longer S1.2.1
- net N$23: now also S1.2, S2.5; no longer S1.2.2, S2.2.1
- net N$24: now also S2.2, S3.5; no longer S2.2.2, S3.2.1
- net N$25: now also S3.2, S4.5; no longer S3.2.2, S4.2.1
- net N$26: now also S4.2, S5.5; no longer S4.2.2, S5.2.1
- net N$27: now also S5.2, S6.5; no longer S5.2.2, S6.2.1
- net N$28: now also S6.2, S7.5; no longer S6.2.2, S7.2.1
- net N$29: now also S7.2, S8.5; no longer S7.2.2, S8.2.1
- net N$30: now also S8.2, S9.5; no longer S8.2.2, S9.2.1
Changed lines of the file:
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@@
 </autorouter>
 <elements>
-<element name="S1" library="switch" package="2P2T" value="2P2T" x="7.62" y="-5.08">
+<element name="S1" library="Menorah" package="JS202011SCQN" value="SWITCH-DPDT" x="7.62" y="-5.08">
 <attribute name="DIGIKEY" value="401-2002-1-ND" x="7.62" y="-5.08" size="1.778" layer="27" display="off"/>
 </element>
@@
 <attribute name="DIGIKEY" value="1276-5502-1-ND" x="-157.48" y="-233.68" size="1.778" layer="27" display="off"/>
 </element>
-<element name="S2" library="switch" package="2P2T" value="2P2T" x="-152.4" y="-242.57">
+<element name="S2" library="Menorah" package="JS202011SCQN" value="SWITCH-DPDT" x="-152.4" y="-242.57">
 <attribute name="DIGIKEY" value="401-2002-1-ND" x="-152.4" y="-242.57" size="1.778" layer="27" display="off"/>
 </element>
-<element name="S3" library="switch" package="2P2T" value="2P2T" x="-152.4" y="-255.27">
+<element name="S3" library="Menorah" package="JS202011SCQN" value="SWITCH-DPDT" x="-152.4" y="-255.27">
 <attribute name="DIGIKEY" value="401-2002-1-ND" x="-152.4" y="-255.27" size="1.778" layer="27" display="off"/>
 </element>
-<element name="S4" library="switch" package="2P2T" value="2P2T" x="-152.4" y="-267.97">
+<element name="S4" library="Menorah" package="JS202011SCQN" value="SWITCH-DPDT" x="-152.4" y="-267.97">
 <attribute name="DIGIKEY" value="401-2002-1-ND" x="-152.4" y="-267.97" size="1.778" layer="27" display="off"/>
 </element>
-<element name="S5" library="switch" package="2P2T" value="2P2T" x="-152.4" y="-280.67">
+<element name="S5" library="Menorah" package="JS202011SCQN" value="SWITCH-DPDT" x="-152.4" y="-280.67">
 <attribute name="DIGIKEY" value="401-2002-1-ND" x="-152.4" y="-280.67" size="1.778" layer="27" display="off"/>
 </element>
-<element name="S6" library="switch" package="2P2T" value="2P2T" x="-152.4" y="-293.37">
+<element name="S6" library="Menorah" package="JS202011SCQN" value="SWITCH-DPDT" x="-152.4" y="-293.37">
 <attribute name="DIGIKEY" value="401-2002-1-ND" x="-152.4" y="-293.37" size="1.778" layer="27" display="off"/>
 </element>
-<element name="S7" library="switch" package="2P2T" value="2P2T" x="-152.4" y="-306.07">
+<element name="S7" library="Menorah" package="JS202011SCQN" value="SWITCH-DPDT" x="-152.4" y="-306.07">
 <attribute name="DIGIKEY" value="401-2002-1-ND" x="-152.4" y="-306.07" size="1.778" layer="27" display="off"/>
 </element>
-<element name="S8" library="switch" package="2P2T" value="2P2T" x="-152.4" y="-318.77">
+<element name="S8" library="Menorah" package="JS202011SCQN" value="SWITCH-DPDT" x="-152.4" y="-318.77">
 <attribute name="DIGIKEY" value="401-2002-1-ND" x="-152.4" y="-318.77" size="1.778" layer="27" display="off"/>
 </element>
-<element name="S9" library="switch" package="2P2T" value="2P2T" x="-152.4" y="-331.47">
+<element name="S9" library="Menorah" package="JS202011SCQN" value="SWITCH-DPDT" x="-152.4" y="-331.47">
 <attribute name="DIGIKEY" value="401-2002-1-ND" x="-152.4" y="-331.47" size="1.778" layer="27" display="off"/>
 </element>
-<element name="S10" library="Menorah" package="KS-01Q-01" value="SWITCH-SPST" x="-153.67" y="-344.17"/>
+<element name="S10" library="Menorah" package="KS-01Q-01" value="SWITCH-SPST" x="-153.67" y="-344.17">
+<attribute name="DIGIKEY" value="EG4791-ND" x="-153.67" y="-344.17" size="1.778" layer="27" display="off"/>
+</element>
 </elements>
 <signals>
@@
 <signal name="N$21">
 <contactref element="IC1" pad="6"/>
-<contactref element="S1" pad="2.1"/>
-<wire x1="7.62" y1="-2.43" x2="-117.475" y2="-177.74" width="0" layer="19" extent="1-1"/>
+<contactref element="S1" pad="5"/>
+<wire x1="7.62" y1="-2.33" x2="-117.475" y2="-177.74" width="0" layer="19" extent="1-1"/>
 </signal>
 <signal name="N$23">
-<contactref element="S1" pad="2.2"/>
-<contactref element="S2" pad="2.1"/>
-<wire x1="7.62" y1="-7.73" x2="-152.4" y2="-239.92" width="0" layer="19" extent="1-1"/>
+<contactref element="S1" pad="2"/>
+<contactref element="S2" pad="5"/>
+<wire x1="7.62" y1="-7.83" x2="-152.4" y2="-239.82" width="0" layer="19" extent="1-1"/>
 </signal>
 <signal name="N$10">
-<contactref element="S1" pad="3.2"/>
+<contactref element="S1" pad="3"/>
 <contactref element="R1" pad="1"/>
-<wire x1="10.62" y1="-7.73" x2="1.59" y2="-116.84" width="0" layer="19" extent="1-1"/>
+<wire x1="10.12" y1="-7.83" x2="1.59" y2="-116.84" width="0" layer="19" extent="1-1"/>
 </signal>
 <signal name="N$11">
 <contactref element="R2" pad="1"/>
-<contactref element="S2" pad="3.2"/>
-<wire x1="-158.43" y1="-195.58" x2="-149.4" y2="-245.22" width="0" layer="19" extent="1-1"/>
+<contactref element="S2" pad="3"/>
+<wire x1="-158.43" y1="-195.58" x2="-149.9" y2="-245.32" width="0" layer="19" extent="1-1"/>
 </signal>
 <signal name="N$12">
 <contactref element="R3" pad="1"/>
-<contactref element="S3" pad="3.2"/>
-<wire x1="-158.43" y1="-201.93" x2="-149.4" y2="-257.92" width="0" layer="19" extent="1-1"/>
+<contactref element="S3" pad="3"/>
+<wire x1="-158.43" y1="-201.93" x2="-149.9" y2="-258.02" width="0" layer="19" extent="1-1"/>
 </signal>
 <signal name="N$13">
 <contactref element="R4" pad="1"/>
-<contactref element="S4" pad="3.2"/>
-<wire x1="-158.43" y1="-208.28" x2="-149.4" y2="-270.62" width="0" layer="19" extent="1-1"/>
+<contactref element="S4" pad="3"/>
+<wire x1="-158.43" y1="-208.28" x2="-149.9" y2="-270.72" width="0" layer="19" extent="1-1"/>
 </signal>
 <signal name="N$14">
 <contactref element="R5" pad="1"/>
-<contactref element="S5" pad="3.2"/>
-<wire x1="-158.43" y1="-214.63" x2="-149.4" y2="-283.32" width="0" layer="19" extent="1-1"/>
+<contactref element="S5" pad="3"/>
+<wire x1="-158.43" y1="-214.63" x2="-149.9" y2="-283.42" width="0" layer="19" extent="1-1"/>
 </signal>
 <signal name="N$15">
 <contactref element="R6" pad="1"/>
-<contactref element="S6" pad="3.2"/>
-<wire x1="-158.43" y1="-220.98" x2="-149.4" y2="-296.02" width="0" layer="19" extent="1-1"/>
+<contactref element="S6" pad="3"/>
+<wire x1="-158.43" y1="-220.98" x2="-149.9" y2="-296.12" width="0" layer="19" extent="1-1"/>
 </signal>
 <signal name="N$16">
 <contactref element="R7" pad="1"/>
-<contactref element="S7" pad="3.2"/>
-<wire x1="-158.43" y1="-227.33" x2="-149.4" y2="-308.72" width="0" layer="19" extent="1-1"/>
+<contactref element="S7" pad="3"/>
+<wire x1="-158.43" y1="-227.33" x2="-149.9" y2="-308.82" width="0" layer="19" extent="1-1"/>
 </signal>
 <signal name="N$17">
 <contactref element="R8" pad="1"/>
-<contactref element="S8" pad="3.2"/>
-<wire x1="-158.43" y1="-233.68" x2="-149.4" y2="-321.42" width="0" layer="19" extent="1-1"/>
+<contactref element="S8" pad="3"/>
+<wire x1="-158.43" y1="-233.68" x2="-149.9" y2="-321.52" width="0" layer="19" extent="1-1"/>
 </signal>
 <signal name="N$18">
 <contactref element="R9" pad="1"/>
-<contactref element="S9" pad="3.2"/>
-<wire x1="-101.28" y1="-157.48" x2="-149.4" y2="-334.12" width="0" layer="19" extent="1-1"/>
+<contactref element="S9" pad="3"/>
+<wire x1="-101.28" y1="-157.48" x2="-149.9" y2="-334.22" width="0" layer="19" extent="1-1"/>
 </signal>
 <signal name="N$24">
-<contactref element="S2" pad="2.2"/>
-<contactref element="S3" pad="2.1"/>
-<wire x1="-152.4" y1="-245.22" x2="-152.4" y2="-252.62" width="0" layer="19" extent="1-1"/>
+<contactref element="S2" pad="2"/>
+<contactref element="S3" pad="5"/>
+<wire x1="-152.4" y1="-245.32" x2="-152.4" y2="-252.52" width="0" layer="19" extent="1-1"/>
 </signal>
 <signal name="N$25">
-<contactref element="S3" pad="2.2"/>
-<contactref element="S4" pad="2.1"/>
-<wire x1="-152.4" y1="-257.92" x2="-152.4" y2="-265.32" width="0" layer="19" extent="1-1"/>
+<contactref element="S3" pad="2"/>
+<contactref element="S4" pad="5"/>
+<wire x1="-152.4" y1="-258.02" x2="-152.4" y2="-265.22" width="0" layer="19" extent="1-1"/>
 </signal>
 <signal name="N$26">
-<contactref element="S4" pad="2.2"/>
-<contactref element="S5" pad="2.1"/>
-<wire x1="-152.4" y1="-270.62" x2="-152.4" y2="-278.02" width="0" layer="19" extent="1-1"/>
+<contactref element="S4" pad="2"/>
+<contactref element="S5" pad="5"/>
+<wire x1="-152.4" y1="-270.72" x2="-152.4" y2="-277.92" width="0" layer="19" extent="1-1"/>
 </signal>
 <signal name="N$27">
-<contactref element="S5" pad="2.2"/>
-<contactref element="S6" pad="2.1"/>
-<wire x1="-152.4" y1="-283.32" x2="-152.4" y2="-290.72" width="0" layer="19" extent="1-1"/>
+<contactref element="S5" pad="2"/>
+<contactref element="S6" pad="5"/>
+<wire x1="-152.4" y1="-283.42" x2="-152.4" y2="-290.62" width="0" layer="19" extent="1-1"/>
 </signal>
 <signal name="N$28">
-<contactref element="S6" pad="2.2"/>
-<contactref element="S7" pad="2.1"/>
-<wire x1="-152.4" y1="-296.02" x2="-152.4" y2="-303.42" width="0" layer="19" extent="1-1"/>
+<contactref element="S6" pad="2"/>
+<contactref element="S7" pad="5"/>
+<wire x1="-152.4" y1="-296.12" x2="-152.4" y2="-303.32" width="0" layer="19" extent="1-1"/>
 </signal>
 <signal name="N$29">
-<contactref element="S7" pad="2.2"/>
-<contactref element="S8" pad="2.1"/>
-<wire x1="-152.4" y1="-308.72" x2="-152.4" y2="-316.12" width="0" layer="19" extent="1-1"/>
+<contactref element="S7" pad="2"/>
+<contactref element="S8" pad="5"/>
+<wire x1="-152.4" y1="-308.82" x2="-152.4" y2="-316.02" width="0" layer="19" extent="1-1"/>
 </signal>
 <signal name="N$30">
-<contactref element="S8" pad="2.2"/>
-<contactref element="S9" pad="2.1"/>
-<wire x1="-152.4" y1="-321.42" x2="-152.4" y2="-328.82" width="0" layer="19" extent="1-1"/>
+<contactref element="S8" pad="2"/>
+<contactref element="S9" pad="5"/>
+<wire x1="-152.4" y1="-321.52" x2="-152.4" y2="-328.72" width="0" layer="19" extent="1-1"/>
 </signal>
 <signal name="+">

Commit message: changed circircuit, updated pcb
Parts:
- removed G1: CR2032, Menorah:BK-913
- removed IC1: (no value), linear:SO08
- removed R12: 100k, rcl:R0805
- added Q1: BUZ382, transistor-fet:TOP3
- R1, R2, R3, R4, R5, R6, R7, R8: value 56 -> 100
- R11: value 51k -> 100
- R9: value 68 -> 100
- moved S10 419.0 mm to (43.3, 25.6)
- moved S9 393.9 mm to (35.0, 15.0), turned to 90 degrees
- moved S8 378.0 mm to (25.0, 15.0), turned to 90 degrees
- moved S7 362.1 mm to (15.0, 15.0), turned to 90 degrees
- moved S5 347.2 mm to (45.0, 5.00), turned to 90 degrees
- moved S6 346.2 mm to (5.00, 15.0), turned to 90 degrees
- moved S4 331.1 mm to (35.0, 5.00), turned to 90 degrees
- moved R8 319.1 mm to (30.0, 24.5), turned to 270 degrees
- moved S3 315.0 mm to (25.0, 5.00), turned to 90 degrees
- moved R7 311.6 mm to (26.0, 24.5), turned to 270 degrees
- moved R6 304.1 mm to (22.0, 24.5), turned to 270 degrees
- moved S2 298.9 mm to (15.0, 5.00), turned to 90 degrees
- moved R5 296.6 mm to (18.0, 24.5), turned to 270 degrees
- moved R4 289.1 mm to (14.0, 24.5), turned to 270 degrees
- moved LED8 288.4 mm to (30.0, 28.7), turned to 180 degrees
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Connections:
- removed net +: G1.+@1
- removed net N$23: S1.2, S2.5
- removed net N$24: S2.2, S3.5
- removed net N$25: S3.2, S4.5
- removed net N$26: S4.2, S5.5
- removed net N$27: S5.2, S6.5
- removed net N$28: S6.2, S7.5
- removed net N$29: S7.2, S8.5
- removed net N$30: S8.2, S9.5
- net N$1: now also LED1.C, R1.1; no longer LED1.A, R1.2
- net N$10: now also R1.2; no longer R1.1
- net N$11: now also R2.2; no longer R2.1
- net N$12: now also R3.2; no longer R3.1
- net N$13: now also R4.2; no longer R4.1
- net N$14: now also R5.2; no longer R5.1
- net N$15: now also R6.2; no longer R6.1
- net N$16: now also R7.2; no longer R7.1
- net N$17: now also R8.2; no longer R8.1
- net N$18: now also R9.2; no longer R9.1
- net N$19: now also R11.2, S10.3, S10.4; no longer IC1.2, R11.1, R12.2
- net N$2: now also LED2.C, R2.1; no longer LED2.A, R2.2
- net N$21: now also Q1.2, S1.2, S2.2, S2.5, S3.2, S3.5, S4.2, S4.5, S5.2, S5.5, S6.2, S6.5, S7.2, S7.5, S8.2, S8.5, S9.2, S9.5; no longer IC1.6
- net N$22: now also Q1.1, R11.1; no longer IC1.3, S10.3, S10.4
- net N$3: now also LED3.C, R3.1; no longer LED3.A, R3.2
- net N$4: now also LED4.C, R4.1; no longer LED4.A, R4.2
- net N$5: now also LED5.C, R5.1; no longer LED5.A, R5.2
- net N$6: now also LED6.C, R6.1; no longer LED6.A, R6.2
- net N$7: now also LED7.C, R7.1; no longer LED7.A, R7.2
- net N$8: now also LED8.C, R8.1; no longer LED8.A, R8.2
- net N$9: now also LED9.C, R9.1; no longer LED9.A, R9.2
- net PE: now also LED1.A, LED2.A, LED3.A, LED4.A, LED5.A, LED6.A, LED7.A, LED8.A, LED9.A, Q1.3; no longer G1.-, IC1.4, LED1.C, LED2.C, LED3.C, LED4.C, LED5.C, LED6.C, LED7.C, LED8.C, LED9.C, R11.2
- net VCC: no longer G1.+, IC1.7, R12.1
Routing:
- net N$21: track 0.00 -> 81.0 mm
- net N$14: track 0.00 -> 42.1 mm, vias 0 -> 2
- net N$13: track 0.00 -> 36.3 mm, vias 0 -> 2
- net N$12: track 0.00 -> 30.0 mm, vias 0 -> 2
- net N$11: track 0.00 -> 25.2 mm, vias 0 -> 2
- net N$15: track 0.00 -> 20.7 mm, vias 0 -> 2
- net N$10: track 0.00 -> 20.4 mm, vias 0 -> 2
- net N$16: track 0.00 -> 14.6 mm, vias 0 -> 2
- net N$18: track 0.00 -> 8.63 mm
- net N$17: track 0.00 -> 7.42 mm, vias 0 -> 2
- net N$8: track 0.00 -> 2.19 mm
- net N$9: track 0.00 -> 2.00 mm
- net N$7: track 0.00 -> 2.00 mm
- net N$6: track 0.00 -> 2.00 mm
- net N$5: track 0.00 -> 2.00 mm
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- added copper zone on layer 16, net PE
Other:
- board size 100 x 80 mm -> 50 x 50 mm

Commit message: design finished
Parts:
- Q1: value BUZ382 -> (none); device transistor-fet:TOP3 -> transistors:SOT-23
- moved R10 50.3 mm to (42.6, 13.9), turned to 0 degrees
- moved Q1 49.8 mm to (42.5, 11.0), turned to 180 degrees
- moved C1 46.7 mm to (42.6, 16.4), turned to 180 degrees
- moved R11 37.4 mm to (43.0, 19.0), turned to 180 degrees
- moved S10 2.00 mm to (43.3, 27.6), turned to 270 degrees
- moved LED8 0.18 mm to (30.0, 28.5)
Connections:
- net N$19: now also S10.2; no longer S10.3
- net N$21: now also Q1.3; no longer Q1.2
- net PE: now also Q1.2; no longer LED1.A, LED2.A, LED3.A, LED4.A, LED5.A, LED6.A, LED7.A, LED8.A, LED9.A, Q1.3
- net VCC: now also LED1.A, LED2.A, LED3.A, LED4.A, LED5.A, LED6.A, LED7.A, LED8.A, LED9.A, S10.3; no longer S10.2
Routing:
- net VCC: track 0.00 -> 67.3 mm, vias 2 -> 4
- net N$21: track 81.0 -> 96.5 mm
- net N$19: track 0.00 -> 11.6 mm
- net N$22: track 0.00 -> 7.18 mm
- net PE: track 0.00 -> 6.87 mm, vias 2 -> 5
- net N$14: track 42.1 -> 44.0 mm
Other:
- board text added: "+"
- board text added: "-"
- board text added: "Alan Rosenthal"
- board text added: "Hanukkah"
- board text added: "Happy"
- board text added: "Nov 10, 2014"
